Commit message: Remove unused inertia to stop rviz warnings

File: urdf/sensors/oem_heading_sensor.xacro (robot description, xacro)
@@ -3,8 +3,4 @@
   <xacro:macro name="oem_heading_sensor" params="name:=heading">
     <link name="${namespace}/${name}">
-      <inertial>
-        <mass value="0.1"/>
-        <inertia ixx="0.000083" ixy="0.0" ixz="0.0" iyy="0.000083" iyz="0.0" izz="0.0125"/>
-      </inertial>
     </link>
     <joint name="${namespace}/${name}_joint" type="revolute">
