Commit message: Fix sensor xacros: joints, parents, and inertials
- GPS: revolute→fixed joint (keep parent=motion_sensor)
- Heading: revolute→fixed, add inertial (keep parent=motion_sensor)
- Radar: uncomment visual geometry, parent→base_link
- Lidar, forward_camera, mbes, pano_array: parent→base_link

Hull-mounted sensors now parent to base_link with positions converted
from MRU-relative to base_link-relative via survey offset properties.
POSMV-mounted sensors (GPS, heading) stay parented to motion_sensor.

Part of #9

File: urdf/sensors/forward_camera.xacro (robot description, xacro)
@@ -38,8 +38,7 @@
     <link name="${namespace}/${name}_optical">
     </link>
-    <!-- Sensor post arm to camera joint -->
-    <joint name="${namespace}/motion_sensor_to_${name}_joint" type="fixed">
+    <joint name="${namespace}/base_link_to_${name}_joint" type="fixed">
       <origin xyz="${x} ${y} ${z}" rpy="${R} ${P} ${Y}" />
-      <parent link="${namespace}/motion_sensor" />
+      <parent link="${namespace}/base_link" />
       <child link="${namespace}/${name}" />
     </joint>

File: urdf/sensors/lidar.xacro (robot description, xacro)
@@ -27,7 +27,7 @@
       </inertial>
     </link>
-    <joint name="${namespace}/motion_sensor_to_${name}_joint" type="fixed">
+    <joint name="${namespace}/base_link_to_${name}_joint" type="fixed">
       <origin xyz="${x} ${y} ${z}" rpy="${R} ${P} ${Y}" />
-      <parent link="${namespace}/motion_sensor" />
+      <parent link="${namespace}/base_link" />
       <child link="${namespace}/${name}" />
     </joint>

File: urdf/sensors/mbes.xacro (robot description, xacro)
@@ -27,7 +27,7 @@
       </inertial>
     </link>
-    <joint name="${namespace}/motion_sensor_to_${name}_joint" type="fixed">
+    <joint name="${namespace}/base_link_to_${name}_joint" type="fixed">
       <origin xyz="${x} ${y} ${z}" rpy="${R} ${P} ${Y}" />
-      <parent link="${namespace}/motion_sensor" />
+      <parent link="${namespace}/base_link" />
       <child link="${namespace}/${name}" />
     </joint>

File: urdf/sensors/oem_gps.xacro (robot description, xacro)
@@ -20,7 +20,5 @@
       </inertial>
     </link>
-    <joint name="${namespace}/${name}_joint" type="revolute">
-      <axis xyz="0 0 1"/>
-      <limit effort="1000.0" lower="0.0" upper="0" velocity="0"/>
+    <joint name="${namespace}/${name}_joint" type="fixed">
       <parent link="${namespace}/motion_sensor" />
       <child link="${namespace}/${name}" />

File: urdf/sensors/oem_heading_sensor.xacro (robot description, xacro)
@@ -3,8 +3,10 @@
   <xacro:macro name="oem_heading_sensor" params="name:=heading">
     <link name="${namespace}/${name}">
+      <inertial>
+        <mass value="0.5"/>
+        <inertia ixx="0.001" ixy="0.0" ixz="0.0" iyy="0.001" iyz="0.0" izz="0.001"/>
+      </inertial>
     </link>
-    <joint name="${namespace}/${name}_joint" type="revolute">
-      <axis xyz="0 0 1"/>
-      <limit effort="1000.0" lower="0.0" upper="0" velocity="0"/>
+    <joint name="${namespace}/${name}_joint" type="fixed">
       <parent link="${namespace}/motion_sensor"/>
       <child link="${namespace}/${name}"/>

File: urdf/sensors/pano_array.xacro (robot description, xacro)
@@ -26,7 +26,7 @@
       </inertial>
     </link>
-    <joint name="${namespace}/motion_sensor_to_${name}_base_joint" type="fixed">
+    <joint name="${namespace}/base_link_to_${name}_joint" type="fixed">
       <origin xyz="${x} ${y} ${z}" rpy="${R} ${P} ${Y}" />
-      <parent link="${namespace}/motion_sensor" />
+      <parent link="${namespace}/base_link" />
       <child link="${namespace}/${name}" />
     </joint>

File: urdf/sensors/radar.xacro (robot description, xacro)
@@ -8,5 +8,5 @@
         <origin xyz="0 0 0" rpy="0 0 0"/>
         <geometry>
-          <!-- <cylinder radius="0.3" length="0.25"/> -->
+          <cylinder radius="0.3" length="0.25"/>
         </geometry>
       </visual>
@@ -27,7 +27,7 @@
       </inertial>
     </link>
-    <joint name="${namespace}/motion_sensor_to_${name}_joint" type="fixed">
+    <joint name="${namespace}/base_link_to_${name}_joint" type="fixed">
       <origin xyz="${x} ${y} ${z}" rpy="${R} ${P} ${Y}" />
-      <parent link="${namespace}/motion_sensor" />
+      <parent link="${namespace}/base_link" />
       <child link="${namespace}/${name}" />
     </joint>
