Commit message: Fix radar geometry to match Simrad Halo 20 dimensions
Cylinder was using placeholder dimensions (r=0.3, h=0.25, m=1kg).
Updated to match actual Halo 20 specs: 510mm diameter, 223mm height,
5.9kg mass with recomputed inertia.

Closes #5

Co-Authored-By: Claude Opus 4.6 <noreply@anthropic.com>

File: urdf/sensors/radar.xacro (robot description, xacro)
@@ -8,18 +8,18 @@
         <origin xyz="0 0 0" rpy="0 0 0"/>
         <geometry>
-          <cylinder radius="0.3" length="0.25"/>
+          <cylinder radius="0.255" length="0.223"/>
         </geometry>
       </visual>
       <collision name="${name}_collision">
         <geometry>
-          <cylinder radius="0.3" length="0.25"/>
+          <cylinder radius="0.255" length="0.223"/>
         </geometry>
       </collision>
       <inertial>
-        <mass value="1"/>
+        <mass value="5.9"/>
         <inertia
-          ixx="0.00109375"
-          iyy="0.00109375"
-          izz="0.00125"
+          ixx="0.12"
+          iyy="0.12"
+          izz="0.096"
           ixy="0"
           ixz="0"

Commit message: refactor(radar): remove visual/collision, keep TF frame only
Hull mesh already includes radar dome visual. Removing the separate
visual and collision geometry avoids visual duplication and prevents
physics issues from collision shapes merging into the hull during
URDF-to-SDF fixed joint conversion.

Closes #5

Co-Authored-By: Claude Code Agent <roland+claude-code@ccom.unh.edu>

File: urdf/sensors/radar.xacro (robot description, xacro)
@@ -4,16 +4,6 @@
                                         x:=0.7 y:=0 z:=1.5
                                         R:=0 P:=0 Y:=0">
+    <!-- TF frame only — hull mesh already includes radar dome visual. -->
     <link name="${namespace}/${name}">
-      <visual name="${name}_visual">
-        <origin xyz="0 0 0" rpy="0 0 0"/>
-        <geometry>
-          <cylinder radius="0.255" length="0.223"/>
-        </geometry>
-      </visual>
-      <collision name="${name}_collision">
-        <geometry>
-          <cylinder radius="0.255" length="0.223"/>
-        </geometry>
-      </collision>
       <inertial>
         <mass value="0.01"/>
