Commit message: Instantiate jetdrive and fix header
- Fix robot name from "wam-v-two-engines" to "ben_jetdrive"
- Change engine parent from motion_sensor to base_link
- Jetdrive is now included and instantiated in ben_mesh.xacro

Part of #9

File: urdf/jetdrive.xacro (robot description, xacro)
@@ -1,4 +1,4 @@
 <?xml version="1.0"?>
-<robot xmlns:xacro="http://ros.org/wiki/xacro" name="wam-v-two-engines">
+<robot xmlns:xacro="http://ros.org/wiki/xacro" name="ben_jetdrive">
   <!-- Macro for inserting an engine with its propeller. -->
   <xacro:macro name="engine" params="prefix position:='0 0 0' orientation:='0 0 0'">
@@ -49,5 +49,5 @@
       <limit lower="${-pi}" upper="${pi}" effort="10" velocity="10"/>
       <origin xyz="${position}" rpy="${orientation}"/>
-      <parent link="${namespace}/motion_sensor"/>
+      <parent link="${namespace}/base_link"/>
       <child link="${prefix}engine_link"/>
     </joint>
