Commit message: Replace wamv_description mesh references with simple geometry
Replace engine mesh with a box (0.2 x 0.15 x 0.6) and propeller mesh
with a cylinder (radius 0.1, length 0.05), removing the dependency on
the wamv_description package from VRX.

Closes #1

Co-Authored-By: Claude Opus 4.6 <noreply@anthropic.com>

File: urdf/jetdrive.xacro (robot description, xacro)
@@ -5,6 +5,7 @@
     <link name="${prefix}engine_link">
       <visual>
+        <origin xyz="-0.16 0 -0.24" rpy="0 0 0" />
         <geometry>
-          <mesh filename="package://wamv_description/models/engine/mesh/engine.dae"/>
+          <box size="0.2 0.15 0.6"/>
         </geometry>
       </visual>
@@ -28,6 +29,7 @@
     <link name="${prefix}propeller_link">
       <visual>
+        <origin xyz="-0.08 0 0" rpy="0 1.57 0" />
         <geometry>
-          <mesh filename="package://wamv_description/models/propeller/mesh/propeller.dae"/>
+          <cylinder radius="0.1" length="0.05"/>
         </geometry>
       </visual>

Commit message: fix(jetdrive): add joint dynamics for Thruster plugin compatibility
Add effort/velocity limits and friction/damping dynamics to the
impeller continuous joint, matching VRX WAM-V thruster configuration.
Required for the Gazebo Thruster plugin to drive the joint.

Closes #5

Co-Authored-By: Claude Code Agent <roland+claude-code@ccom.unh.edu>

File: urdf/jetdrive.xacro (robot description, xacro)
@@ -46,4 +46,6 @@
       <child link="${namespace}/${name}_impeller"/>
       <axis xyz="1 0 0"/>
+      <limit effort="100" velocity="100"/>
+      <dynamics friction="0.05" damping="0.05"/>
     </joint>
   </xacro:macro>

Commit message: fix: use xacro radians() for deflector limits and update rviz frames
Replace hard-coded ±0.524 rad with ${-radians(30)}/${radians(30)} in
jetdrive.xacro for clarity. Update urdf.rviz to reference the new
jetdrive and mbes_ram frame names introduced in the waterjet commit.

Co-Authored-By: Claude Opus 4.6 <noreply@anthropic.com>

File: urdf/jetdrive.xacro (robot description, xacro)
@@ -31,5 +31,5 @@
       <child link="${namespace}/${name}_deflector"/>
       <axis xyz="0 0 1"/>
-      <limit lower="-0.524" upper="0.524" effort="100" velocity="1.0"/>
+      <limit lower="${-radians(30)}" upper="${radians(30)}" effort="100" velocity="1.0"/>
     </joint>
     <!-- Impeller — spins to generate thrust force -->
