Commit message: Fix hull mass properties and inertia for stable Gazebo simulation
Update hull mass to 883 kg and CG to z=0.186 per ASV GA drawing
(ASV-396-7-000-i0001-01). Replace unreliable OnShape inertia with
uniform box estimate (4.17m x 1.58m x 0.63m) and zero off-diagonal
products — the OnShape values caused roll-yaw cross-coupling that
capsized the hull when amplified by sensor-mass merging during
URDF-to-SDF fixed joint conversion.

Reduce sensor link masses to 0.01 kg (reference frames only; total
displacement is accounted for in hull_mass). Fix engine joints to
type=fixed and remove engine collision geometry — BEN uses an
Alamarin-Jet AJ 160 waterjet, not a steerable outboard.

Co-Authored-By: Claude Opus 4.6 <noreply@anthropic.com>

File: urdf/ben_mesh.xacro (robot description, xacro)
@@ -8,15 +8,22 @@
        Source: OnShape CAD model
        ============================================================ -->
-  <!-- Hull mass properties (from OnShape) -->
-  <xacro:property name="hull_mass" value="950" />
+  <!-- Hull mass properties.
+       GA drawing (ASV-396-7-000-i0001-01): 883 kg displacement, 0.40m draft.
+       CG lowered from OnShape estimate to ~60% of draft above keel for
+       typical monohull stability. In base_link frame CG_z = 0.186. -->
+  <xacro:property name="hull_mass" value="883" />
   <xacro:property name="cg_x" value="-0.911" />
   <xacro:property name="cg_y" value="-0.018" />
-  <xacro:property name="cg_z" value="-0.182" />
-  <xacro:property name="ixx" value="280.97548467" />
-  <xacro:property name="ixy" value="-9.237803" />
-  <xacro:property name="ixz" value="-2.02566202" />
-  <xacro:property name="iyy" value="866.01489076" />
-  <xacro:property name="iyz" value="-0.43969229" />
-  <xacro:property name="izz" value="793.7913527" />
+  <xacro:property name="cg_z" value="-0.346" />
+  <!-- Inertia estimated as uniform-density box from GA drawing dimensions
+       (4.17m x 1.58m x 0.63m at 883 kg). OnShape CAD values were unreliable
+       and off-diagonal products caused capsizing when amplified by sensor-mass
+       merging during URDF-to-SDF fixed joint conversion. -->
+  <xacro:property name="ixx" value="212.9" />
+  <xacro:property name="ixy" value="0.0" />
+  <xacro:property name="ixz" value="0.0" />
+  <xacro:property name="iyy" value="1308.7" />
+  <xacro:property name="iyz" value="0.0" />
+  <xacro:property name="izz" value="1463.2" />
   <!-- POSMV MRU location relative to base_link.
        The visual/collision meshes were authored with their origin at this point,
@@ -97,6 +104,8 @@
   <link name="${namespace}/motion_sensor">
     <inertial>
-      <mass value="5.0"/>
-      <inertia ixx="0.01" ixy="0.0" ixz="0.0" iyy="0.01" iyz="0.0" izz="0.01"/>
+      <!-- Near-zero mass: sensor link is a reference frame only.
+           Total displacement (883 kg) is accounted for in hull_mass. -->
+      <mass value="0.01"/>
+      <inertia ixx="0.0001" ixy="0.0" ixz="0.0" iyy="0.0001" iyz="0.0" izz="0.0001"/>
     </inertial>
   </link>

File: urdf/jetdrive.xacro (robot description, xacro)
@@ -10,19 +10,10 @@
         </geometry>
       </visual>
-      <collision name="${prefix}engine_vertical_axis_collision">
-        <origin xyz="-0.16 0 -0.24" rpy="0 0 0" />
-        <geometry>
-          <box size="0.2 0.15 0.83" />
-        </geometry>
-      </collision>
-      <collision name="${prefix}engine_rear_end_collision">
-        <origin xyz="-0.34 0 0.12" rpy="0 0 0" />
-        <geometry>
-          <box size="0.12 0.15 0.12" />
-        </geometry>
-      </collision>
+      <!-- No collision — engine is internal (Alamarin-Jet AJ 160 waterjet).
+           Collision geometries inside the hull mesh cause physics issues
+           when fixed joints are merged during URDF-to-SDF conversion. -->
       <inertial>
-        <mass value="15"/>
-        <inertia ixx="0.889245" ixy="0.0" ixz="0.0" iyy="0.911125" iyz="0.0" izz="0.078125"/>
+        <mass value="0.01"/>
+        <inertia ixx="0.0001" ixy="0.0" ixz="0.0" iyy="0.0001" iyz="0.0" izz="0.0001"/>
       </inertial>
     </link>
@@ -34,29 +25,23 @@
         </geometry>
       </visual>
-      <collision name="${prefix}propeller_collision">
-        <origin xyz="-0.08 0 0" rpy="0 1.57 0" />
-        <geometry>
-          <cylinder length="0.18" radius="0.24" />
-        </geometry>
-      </collision>
+      <!-- No collision — internal waterjet impeller -->
       <inertial>
-        <mass value="0.5"/>
-        <inertia ixx="0.008545" ixy="0.0" ixz="0.0" iyy="0.008545" iyz="0.0" izz="0.0144"/>
+        <mass value="0.01"/>
+        <inertia ixx="0.0001" ixy="0.0" ixz="0.0" iyy="0.0001" iyz="0.0" izz="0.0001"/>
       </inertial>
     </link>
-    <joint name="${prefix}chasis_engine_joint" type="revolute">
-      <axis xyz="0 0 1"/>
-      <limit lower="${-pi}" upper="${pi}" effort="10" velocity="10"/>
+    <!-- Both joints fixed: BEN uses an Alamarin-Jet AJ 160 waterjet,
+         not a steerable outboard. The revolute/continuous joints were
+         placeholders from the ROS 2 port. Fixing them until a proper
+         waterjet model is implemented. -->
+    <joint name="${prefix}chasis_engine_joint" type="fixed">
       <origin xyz="${position}" rpy="${orientation}"/>
       <parent link="${namespace}/base_link"/>
       <child link="${prefix}engine_link"/>
     </joint>
-    <joint name="${prefix}engine_propeller_joint" type="continuous">
-      <axis rpy="0 0 0" xyz="1 0 0"/>
+    <joint name="${prefix}engine_propeller_joint" type="fixed">
       <parent link="${prefix}engine_link"/>
       <child link="${prefix}propeller_link"/>
       <origin rpy="0 0 0" xyz="-0.278156 0 -0.509371"/>
-      <limit effort="100" velocity="100" />
-      <dynamics friction="0.05" damping="0.05" />
     </joint>
   </xacro:macro>

File: urdf/sensors/forward_camera.xacro (robot description, xacro)
@@ -24,9 +24,9 @@
       <!-- Model inertia as box with <size>0.078 0.03 0.03</size> -->
       <inertial>
-        <mass value="0.3"/>
+        <mass value="0.01"/>
         <inertia
-          ixx="0.0000450"
-          iyy="0.0001746"
-          izz="0.0001746"
+          ixx="0.0001"
+          iyy="0.0001"
+          izz="0.0001"
           ixy="0"
           ixz="0"

File: urdf/sensors/lidar.xacro (robot description, xacro)
@@ -17,9 +17,9 @@
       </collision>
       <inertial>
-        <mass value="1"/>
+        <mass value="0.01"/>
         <inertia
-          ixx="0.00109375"
-          iyy="0.00109375"
-          izz="0.00125"
+          ixx="0.0001"
+          iyy="0.0001"
+          izz="0.0001"
           ixy="0"
           ixz="0"

File: urdf/sensors/mbes.xacro (robot description, xacro)
@@ -17,9 +17,9 @@
       </collision>
       <inertial>
-        <mass value="1"/>
+        <mass value="0.01"/>
         <inertia
-          ixx="0.00109375"
-          iyy="0.00109375"
-          izz="0.00125"
+          ixx="0.0001"
+          iyy="0.0001"
+          izz="0.0001"
           ixy="0"
           ixz="0"

File: urdf/sensors/oem_gps.xacro (robot description, xacro)
@@ -16,6 +16,6 @@
       </collision>
       <inertial>
-        <mass value="1"/>
-        <inertia ixx="0.006458" ixy="0.0" ixz="0.0" iyy="0.006458" iyz="0.0" izz="0.01125"/>
+        <mass value="0.01"/>
+        <inertia ixx="0.0001" ixy="0.0" ixz="0.0" iyy="0.0001" iyz="0.0" izz="0.0001"/>
       </inertial>
     </link>

File: urdf/sensors/oem_heading_sensor.xacro (robot description, xacro)
@@ -4,6 +4,6 @@
     <link name="${namespace}/${name}">
       <inertial>
-        <mass value="0.5"/>
-        <inertia ixx="0.001" ixy="0.0" ixz="0.0" iyy="0.001" iyz="0.0" izz="0.001"/>
+        <mass value="0.01"/>
+        <inertia ixx="0.0001" ixy="0.0" ixz="0.0" iyy="0.0001" iyz="0.0" izz="0.0001"/>
       </inertial>
     </link>

File: urdf/sensors/pano_array.xacro (robot description, xacro)
@@ -16,9 +16,9 @@
       </collision>
       <inertial>
-        <mass value="0.3"/>
+        <mass value="0.01"/>
         <inertia
-          ixx="0.0000450"
-          iyy="0.0001746"
-          izz="0.0001746"
+          ixx="0.0001"
+          iyy="0.0001"
+          izz="0.0001"
           ixy="0"
           ixz="0"

File: urdf/sensors/pano_camera.xacro (robot description, xacro)
@@ -18,9 +18,9 @@
       <!-- Model inertia as box with <size>0.078 0.03 0.03</size> -->
       <inertial>
-        <mass value="0.3"/>
+        <mass value="0.01"/>
         <inertia
-          ixx="0.0000450"
-          iyy="0.0001746"
-          izz="0.0001746"
+          ixx="0.0001"
+          iyy="0.0001"
+          izz="0.0001"
           ixy="0"
           ixz="0"

File: urdf/sensors/radar.xacro (robot description, xacro)
@@ -17,9 +17,9 @@
       </collision>
       <inertial>
-        <mass value="5.9"/>
+        <mass value="0.01"/>
         <inertia
-          ixx="0.12"
-          iyy="0.12"
-          izz="0.096"
+          ixx="0.0001"
+          iyy="0.0001"
+          izz="0.0001"
           ixy="0"
           ixz="0"

Commit message: feat: waterjet propulsion model and MBES retractable ram
Replace engine/propeller model with Alamarin-Jet AJ 160 waterjet:
- jetdrive_mount (fixed) → deflector (revolute ±30°) → impeller (continuous)
- Deflector/bucket redirects jet for steering, impeller spins for thrust

Replace static MBES with retractable ram model:
- Prismatic joint (Z axis, 0 to -226mm travel) for Kongsberg EM 2040P
- MBES transducer as TF frame only (hull mesh has visual)
- 180° roll on MBES frame for downward-facing convention

Update ben_mesh.xacro with new macro names and positions.
All non-base_link masses 0.01 kg to prevent inertia cross-coupling.

Closes #5

Co-Authored-By: Claude Code Agent <roland+claude-code@ccom.unh.edu>

File: urdf/ben_mesh.xacro (robot description, xacro)
@@ -53,8 +53,8 @@
   <xacro:property name="forward_camera_y" value="0.1" />
   <xacro:property name="forward_camera_z" value="0.742" />
-  <!-- MBES (hull-mounted, relative to MRU) -->
-  <xacro:property name="mbes_x" value="0.0" />
+  <!-- MBES (hull-mounted, on retractable ram, relative to MRU) -->
+  <xacro:property name="mbes_x" value="-0.5" />
   <xacro:property name="mbes_y" value="0.0" />
-  <xacro:property name="mbes_z" value="-1.0" />
+  <xacro:property name="mbes_z" value="-0.4" />
   <!-- GPS (POSMV-mounted, relative to motion_sensor) -->
   <xacro:property name="gps_x" value="-0.953" />
@@ -62,8 +62,8 @@
   <xacro:property name="gps_z" value="0.628" />
   <!-- Heading sensor at motion_sensor origin (no offset) -->
-  <!-- Jetdrive engine (hull-mounted, relative to MRU) -->
-  <xacro:property name="engine_x" value="-1.6" />
-  <xacro:property name="engine_y" value="0.0" />
-  <xacro:property name="engine_z" value="-0.35" />
+  <!-- Jetdrive (stern, hull-mounted, relative to MRU) -->
+  <xacro:property name="jetdrive_x" value="-1.1" />
+  <xacro:property name="jetdrive_y" value="0.0" />
+  <xacro:property name="jetdrive_z" value="-0.1" />
   <!-- ============================================================
        End of survey offsets
@@ -125,6 +125,5 @@
   <xacro:include filename="$(find ben_description)/urdf/sensors/mbes.xacro" />
   <xacro:ben_mbes name="mbes"
-    x="${mru_x + mbes_x}" y="${mru_y + mbes_y}" z="${mru_z + mbes_z}"
-    R="${radians(180)}"/>
+    x="${mru_x + mbes_x}" y="${mru_y + mbes_y}" z="${mru_z + mbes_z}"/>
   <!-- POSMV-mounted sensors (positions relative to motion_sensor) -->
   <xacro:include filename="$(find ben_description)/urdf/sensors/oem_gps.xacro" />
@@ -132,7 +131,7 @@
   <xacro:include filename="$(find ben_description)/urdf/sensors/oem_heading_sensor.xacro" />
   <xacro:oem_heading_sensor name="heading"/>
-  <!-- Jetdrive -->
+  <!-- Jetdrive (Alamarin-Jet AJ 160 waterjet) -->
   <xacro:include filename="$(find ben_description)/urdf/jetdrive.xacro" />
-  <xacro:engine prefix="${namespace}/"
-    position="${mru_x + engine_x} ${mru_y + engine_y} ${mru_z + engine_z}"/>
+  <xacro:ben_jetdrive name="jetdrive"
+    x="${mru_x + jetdrive_x}" y="${mru_y + jetdrive_y}" z="${mru_z + jetdrive_z}"/>
 </robot>

File: urdf/jetdrive.xacro (robot description, xacro)
@@ -1,47 +1,49 @@
 <?xml version="1.0"?>
-<robot xmlns:xacro="http://ros.org/wiki/xacro" name="ben_jetdrive">
-  <!-- Macro for inserting an engine with its propeller. -->
-  <xacro:macro name="engine" params="prefix position:='0 0 0' orientation:='0 0 0'">
-    <link name="${prefix}engine_link">
-      <visual>
-        <origin xyz="-0.16 0 -0.24" rpy="0 0 0" />
-        <geometry>
-          <box size="0.2 0.15 0.6"/>
-        </geometry>
-      </visual>
-      <!-- No collision — engine is internal (Alamarin-Jet AJ 160 waterjet).
-           Collision geometries inside the hull mesh cause physics issues
-           when fixed joints are merged during URDF-to-SDF conversion. -->
+<robot xmlns:xacro="http://ros.org/wiki/xacro">
+  <!-- Alamarin-Jet AJ 160 waterjet model.
+       Internal waterjet with deflector/bucket for steering and reverse.
+       No visual/collision — the jet is inside the hull. -->
+  <xacro:macro name="ben_jetdrive" params="name x:=0 y:=0 z:=0">
+    <!-- Mount point (fixed to hull, no visual/collision) -->
+    <link name="${namespace}/${name}_mount">
       <inertial>
         <mass value="0.01"/>
-        <inertia ixx="0.0001" ixy="0.0" ixz="0.0" iyy="0.0001" iyz="0.0" izz="0.0001"/>
+        <inertia ixx="0.0001" ixy="0.0" ixz="0.0"
+                 iyy="0.0001" iyz="0.0" izz="0.0001"/>
       </inertial>
     </link>
-    <link name="${prefix}propeller_link">
-      <visual>
-        <origin xyz="-0.08 0 0" rpy="0 1.57 0" />
-        <geometry>
-          <cylinder radius="0.1" length="0.05"/>
-        </geometry>
-      </visual>
-      <!-- No collision — internal waterjet impeller -->
+    <joint name="${namespace}/${name}_mount_joint" type="fixed">
+      <origin xyz="${x} ${y} ${z}" rpy="0 0 0"/>
+      <parent link="${namespace}/base_link"/>
+      <child link="${namespace}/${name}_mount"/>
+    </joint>
+    <!-- Deflector/bucket — redirects jet for steering (yaw ±30°) -->
+    <link name="${namespace}/${name}_deflector">
       <inertial>
         <mass value="0.01"/>
-        <inertia ixx="0.0001" ixy="0.0" ixz="0.0" iyy="0.0001" iyz="0.0" izz="0.0001"/>
+        <inertia ixx="0.0001" ixy="0.0" ixz="0.0"
+                 iyy="0.0001" iyz="0.0" izz="0.0001"/>
       </inertial>
     </link>
-    <!-- Both joints fixed: BEN uses an Alamarin-Jet AJ 160 waterjet,
-         not a steerable outboard. The revolute/continuous joints were
-         placeholders from the ROS 2 port. Fixing them until a proper
-         waterjet model is implemented. -->
-    <joint name="${prefix}chasis_engine_joint" type="fixed">
-      <origin xyz="${position}" rpy="${orientation}"/>
-      <parent link="${namespace}/base_link"/>
-      <child link="${prefix}engine_link"/>
+    <joint name="${namespace}/${name}_deflector_joint" type="revolute">
+      <origin xyz="0 0 0" rpy="0 0 0"/>
+      <parent link="${namespace}/${name}_mount"/>
+      <child link="${namespace}/${name}_deflector"/>
+      <axis xyz="0 0 1"/>
+      <limit lower="-0.524" upper="0.524" effort="100" velocity="1.0"/>
     </joint>
-    <joint name="${prefix}engine_propeller_joint" type="fixed">
-      <parent link="${prefix}engine_link"/>
-      <child link="${prefix}propeller_link"/>
-      <origin rpy="0 0 0" xyz="-0.278156 0 -0.509371"/>
+    <!-- Impeller — spins to generate thrust force -->
+    <link name="${namespace}/${name}_impeller">
+      <inertial>
+        <mass value="0.01"/>
+        <inertia ixx="0.0001" ixy="0.0" ixz="0.0"
+                 iyy="0.0001" iyz="0.0" izz="0.0001"/>
+      </inertial>
+    </link>
+    <joint name="${namespace}/${name}_impeller_joint" type="continuous">
+      <origin xyz="0 0 0" rpy="0 0 0"/>
+      <parent link="${namespace}/${name}_deflector"/>
+      <child link="${namespace}/${name}_impeller"/>
+      <axis xyz="1 0 0"/>
     </joint>
   </xacro:macro>

File: urdf/sensors/mbes.xacro (robot description, xacro)
@@ -1,34 +1,35 @@
 <?xml version="1.0" encoding="UTF-8"?>
 <robot xmlns:xacro="http://ros.org/wiki/xacro">
-  <xacro:macro name="ben_mbes" params="name
-                                        x:=0.0 y:=0.0 z:=-1.0
-                                        R:=3.14 P:=0 Y:=0">
-    <link name="${namespace}/${name}">
-      <visual name="${name}_visual">
-        <origin xyz="0 0 0" rpy="0 0 0"/>
-        <geometry>
-          <cylinder radius="0.3" length="0.25"/>
-        </geometry>
-      </visual>
-      <collision name="${name}_collision">
-        <geometry>
-          <cylinder radius="0.3" length="0.25"/>
-        </geometry>
-      </collision>
+  <!-- Kongsberg EM 2040P MBES on retractable ram.
+       Travel = max_draft(630mm) - hull_draft(404mm) = 226mm downward.
+       No visual/collision — hull mesh includes the ram housing. -->
+  <xacro:macro name="ben_mbes" params="name x:=0 y:=0 z:=0">
+    <!-- Ram — prismatic joint for vertical travel (0 to -0.226 m) -->
+    <link name="${namespace}/${name}_ram">
       <inertial>
         <mass value="0.01"/>
-        <inertia
-          ixx="0.0001"
-          iyy="0.0001"
-          izz="0.0001"
-          ixy="0"
-          ixz="0"
-          iyz="0"/>
+        <inertia ixx="0.0001" ixy="0.0" ixz="0.0"
+                 iyy="0.0001" iyz="0.0" izz="0.0001"/>
       </inertial>
     </link>
-    <joint name="${namespace}/base_link_to_${name}_joint" type="fixed">
-      <origin xyz="${x} ${y} ${z}" rpy="${R} ${P} ${Y}" />
-      <parent link="${namespace}/base_link" />
-      <child link="${namespace}/${name}" />
+    <joint name="${namespace}/${name}_ram_joint" type="prismatic">
+      <origin xyz="${x} ${y} ${z}" rpy="0 0 0"/>
+      <parent link="${namespace}/base_link"/>
+      <child link="${namespace}/${name}_ram"/>
+      <axis xyz="0 0 1"/>
+      <limit lower="-0.226" upper="0.0" effort="100" velocity="0.05"/>
+    </joint>
+    <!-- MBES transducer — TF frame only (like radar) -->
+    <link name="${namespace}/${name}">
+      <inertial>
+        <mass value="0.01"/>
+        <inertia ixx="0.0001" ixy="0.0" ixz="0.0"
+                 iyy="0.0001" iyz="0.0" izz="0.0001"/>
+      </inertial>
+    </link>
+    <joint name="${namespace}/${name}_joint" type="fixed">
+      <origin xyz="0 0 0" rpy="${radians(180)} 0 0"/>
+      <parent link="${namespace}/${name}_ram"/>
+      <child link="${namespace}/${name}"/>
     </joint>
   </xacro:macro>
