Commit message: Restructure hull: move content to base_link, add survey offsets
Move mass, visual, collision, and inertial from motion_sensor to
base_link. Add centralized survey offsets block with all physical
measurements. Replace degenerate BEN_convex_hull.dae (8578 vertices,
947 degenerate faces) with low-poly convex hull STL (319 vertices,
634 faces, watertight). Keep motion_sensor as POSMV MRU reference
frame with lightweight inertial.

Closes #5 (empty radar geometry — fixed in radar.xacro)
Closes #6 (missing heading inertial — fixed in oem_heading_sensor.xacro)
Part of #9

File: urdf/ben_mesh.xacro (robot description, xacro)
@@ -3,5 +3,11 @@
   <xacro:arg name="namespace" default="ben"/>
   <xacro:property name="namespace" value="$(arg namespace)" scope="global" />
-  <xacro:property name="mass" value="950" />
+  <!-- ============================================================
+       Survey offsets — UPDATE THIS SECTION AFTER RESURVEY
+       All positions in meters.
+       Source: OnShape CAD model
+       ============================================================ -->
+  <!-- Hull mass properties (from OnShape) -->
+  <xacro:property name="hull_mass" value="950" />
   <xacro:property name="cg_x" value="-0.911" />
   <xacro:property name="cg_y" value="-0.018" />
@@ -13,59 +19,111 @@
   <xacro:property name="iyz" value="-0.43969229" />
   <xacro:property name="izz" value="793.7913527" />
-  <xacro:property name="buoyancy_offset" value=".35" />
+  <!-- POSMV MRU location relative to base_link.
+       The visual/collision meshes were authored with their origin at this point,
+       so the mesh geometry <origin> uses the same offset. -->
+  <xacro:property name="mru_x" value="0.911" />
+  <xacro:property name="mru_y" value="0.018" />
+  <xacro:property name="mru_z" value="0.532" />
+  <!-- Sensor positions, measured relative to the POSMV MRU reference point.
+       Hull-mounted sensors are parented to base_link in the URDF, so their
+       joint origins add the MRU offset (e.g. x="${mru_x + lidar_x}").
+       POSMV-mounted sensors (gps, heading) are parented to motion_sensor
+       and use these offsets directly. -->
+  <!-- Lidar (hull-mounted, relative to MRU) -->
+  <xacro:property name="lidar_x" value="-1.98" />
+  <xacro:property name="lidar_y" value="0.0" />
+  <xacro:property name="lidar_z" value="1.403" />
+  <!-- Radar (hull-mounted, relative to MRU) -->
+  <xacro:property name="radar_x" value="-1.8" />
+  <xacro:property name="radar_y" value="0.0" />
+  <xacro:property name="radar_z" value="1.3" />
+  <!-- Panoramic camera array (hull-mounted, relative to MRU) -->
+  <xacro:property name="pano_x" value="-1.98" />
+  <xacro:property name="pano_y" value="0.0" />
+  <xacro:property name="pano_z" value="1.266" />
+  <!-- Forward camera (hull-mounted, relative to MRU) -->
+  <xacro:property name="forward_camera_x" value="-1.307" />
+  <xacro:property name="forward_camera_y" value="0.1" />
+  <xacro:property name="forward_camera_z" value="0.742" />
+  <!-- MBES (hull-mounted, relative to MRU) -->
+  <xacro:property name="mbes_x" value="0.0" />
+  <xacro:property name="mbes_y" value="0.0" />
+  <xacro:property name="mbes_z" value="-1.0" />
+  <!-- GPS (POSMV-mounted, relative to motion_sensor) -->
+  <xacro:property name="gps_x" value="-0.953" />
+  <xacro:property name="gps_y" value="0.103" />
+  <xacro:property name="gps_z" value="0.628" />
+  <!-- Heading sensor at motion_sensor origin (no offset) -->
+  <!-- Jetdrive engine (hull-mounted, relative to MRU) -->
+  <xacro:property name="engine_x" value="-1.6" />
+  <xacro:property name="engine_y" value="0.0" />
+  <xacro:property name="engine_z" value="-0.35" />
+  <!-- ============================================================
+       End of survey offsets
+       ============================================================ -->
+  <!-- base_link: hull frame at waterline reference.
+       All hull-mounted sensors and the visual/collision mesh attach here. -->
   <link name="${namespace}/base_link">
+    <visual>
+      <!-- Mesh origin is at the POSMV MRU location -->
+      <origin xyz="${mru_x} ${mru_y} ${mru_z}" rpy="0 0 0"/>
+      <geometry>
+        <mesh filename="package://ben_description/models/meshes/BEN_shell.dae"/>
+      </geometry>
+    </visual>
+    <collision>
+      <origin xyz="${mru_x} ${mru_y} ${mru_z}" rpy="0 0 0"/>
+      <geometry>
+        <mesh filename="package://ben_description/models/meshes/BEN_shell_collision.stl"/>
+      </geometry>
+    </collision>
+    <inertial>
+      <!-- CG in base_link frame = MRU offset + CG relative to MRU -->
+      <origin xyz="${mru_x + cg_x} ${mru_y + cg_y} ${mru_z + cg_z}" rpy="0 0 0"/>
+      <mass value="${hull_mass}"/>
+      <inertia
+        ixx="${ixx}" ixy="${ixy}" ixz="${ixz}"
+        iyy="${iyy}" iyz="${iyz}"
+        izz="${izz}"/>
+    </inertial>
   </link>
-  <joint name="${namespace}_base_to_motion_sensor_joint" type="fixed">
-      <parent link="${namespace}/base_link"/>
-      <child link="${namespace}/motion_sensor"/>
-      <origin xyz="${- cg_x} ${- cg_y} ${buoyancy_offset - cg_z}" rpy="0 0 0"/>
+  <!-- motion_sensor: POSMV MRU physical reference frame.
+       GPS and heading sensor are parented here. -->
+  <joint name="${namespace}/base_link_to_motion_sensor_joint" type="fixed">
+    <parent link="${namespace}/base_link"/>
+    <child link="${namespace}/motion_sensor"/>
+    <origin xyz="${mru_x} ${mru_y} ${mru_z}" rpy="0 0 0"/>
   </joint>
   <link name="${namespace}/motion_sensor">
-    <visual>
-        <geometry>
-            <mesh filename="package://ben_description/models/meshes/BEN_shell.dae"/>
-        </geometry>
-    </visual>
-    <!-- footprint 2.65, 0
-                    2.6,  0.1
-                    2.4,  0.4
-                    1.9,  0.6
-                    1.0,  0.85
-                    -1.3, 0.85
-                    -1.35, 0.4
-                    -1.6, 0.35
-                    (repeat symetrically for other side)
-                    (Meters relative to base frame)
-                     -->
-    <collision>
-        <geometry>
-            <mesh filename="package://ben_description/models/meshes/BEN_convex_hull.dae"/>
-        </geometry>
-    </collision>
     <inertial>
-        <!--Values obtained from OnShape-->
-        <origin xyz="${cg_x} ${cg_y} ${cg_z}" rpy="0 0 0"/>
-        <mass value="${mass}"/>
-        <inertia
-            ixx="${ixx}" ixy="${ixy}" ixz="${ixz}"
-            iyy="${iyy}" iyz="${iyz}"
-            izz="${izz}"/>
+      <mass value="5.0"/>
+      <inertia ixx="0.01" ixy="0.0" ixz="0.0" iyy="0.01" iyz="0.0" izz="0.01"/>
     </inertial>
   </link>
+  <!-- Hull-mounted sensors (positions converted from MRU-relative to base_link-relative) -->
   <xacro:include filename="$(find ben_description)/urdf/sensors/lidar.xacro" />
-  <xacro:ben_lidar name="lidar" x="-1.98" y="0.0" z="1.403"/>
+  <xacro:ben_lidar name="lidar"
+    x="${mru_x + lidar_x}" y="${mru_y + lidar_y}" z="${mru_z + lidar_z}"/>
   <xacro:include filename="$(find ben_description)/urdf/sensors/radar.xacro" />
-  <xacro:ben_radar name="radar" x="-1.8" y="0.0" z="1.3"/>
+  <xacro:ben_radar name="radar"
+    x="${mru_x + radar_x}" y="${mru_y + radar_y}" z="${mru_z + radar_z}"/>
   <xacro:include filename="$(find ben_description)/urdf/sensors/pano_array.xacro" />
-  <xacro:pano_array name="pano" x="-1.98" z="1.266"/>
-  <!-- HACK moved pano array up so light is not in field of view -->
-  <!-- <xacro:pano_array name="pano" x="-1.98" z="1.366"/>   -->
+  <xacro:pano_array name="pano"
+    x="${mru_x + pano_x}" y="${mru_y + pano_y}" z="${mru_z + pano_z}"/>
+  <xacro:include filename="$(find ben_description)/urdf/sensors/forward_camera.xacro" />
+  <xacro:forward_camera name="forward_camera"
+    x="${mru_x + forward_camera_x}" y="${mru_y + forward_camera_y}" z="${mru_z + forward_camera_z}"/>
+  <xacro:include filename="$(find ben_description)/urdf/sensors/mbes.xacro" />
+  <xacro:ben_mbes name="mbes"
+    x="${mru_x + mbes_x}" y="${mru_y + mbes_y}" z="${mru_z + mbes_z}"
+    R="${radians(180)}"/>
+  <!-- POSMV-mounted sensors (positions relative to motion_sensor) -->
   <xacro:include filename="$(find ben_description)/urdf/sensors/oem_gps.xacro" />
-  <xacro:oem_gps name="gps" x="-0.953" y="0.103" z="0.628"/>
+  <xacro:oem_gps name="gps" x="${gps_x}" y="${gps_y}" z="${gps_z}"/>
   <xacro:include filename="$(find ben_description)/urdf/sensors/oem_heading_sensor.xacro" />
   <xacro:oem_heading_sensor name="heading"/>
-  <xacro:include filename="$(find ben_description)/urdf/sensors/forward_camera.xacro" />
-  <xacro:forward_camera name="forward_camera" y="0.1" x="-1.307" z="0.742" P="${radians(0)}" />
-  <xacro:include filename="$(find ben_description)/urdf/sensors/mbes.xacro" />
-  <xacro:ben_mbes name="mbes" />
+  <!-- Jetdrive -->
+  <xacro:include filename="$(find ben_description)/urdf/jetdrive.xacro" />
+  <xacro:engine prefix="${namespace}/"
+    position="${mru_x + engine_x} ${mru_y + engine_y} ${mru_z + engine_z}"/>
 </robot>

Commit message: Add Garmin sidescan TF frames (placeholder geometry) (closes #13)
Add TF frames so the garmin_sidescan driver's per-channel frame_ids resolve in
the tree. Mounting/orientation lives in TF, not driver params.

- New urdf/sensors/garmin_sidescan.xacro (ben_garmin_sidescan macro): a mount
  frame plus _down / _port / _starboard channel frames (TF-only, like radar).
  Range axis = each frame's local +Z (rviz_sonar_image places a fixed beam's
  samples along +Z): _down faces down (like the MBES), _port/_starboard fire to
  the sides. Side-scan grazing tilt is a 0 placeholder, to be calibrated.
- Instantiate in ben_mesh.xacro, anchored to the MBES: 0.5 m forward, glued to
  the hull (z = mbes_z - 0.01). Placeholder per operator description.

Frames are named garmin_sidescan(_port/_starboard/_down), not "gcv" -- the
device name is obscure; descriptive identifiers everywhere, "GCV-20" only in
comments.

Part of the BizzyBoat Garmin sidescan wiring (driver: marine_tools#17).

File: urdf/ben_mesh.xacro (robot description, xacro)
@@ -57,4 +57,11 @@
   <xacro:property name="mbes_y" value="0.0" />
   <xacro:property name="mbes_z" value="-0.4" />
+  <!-- Garmin GCV-20 sidescan (hull-mounted, relative to MRU).
+       PLACEHOLDER: ~0.5 m forward of the MBES, glued to the hull with the
+       transducer faces ~1 cm below it. Anchored to the MBES offsets so it
+       tracks the same hull reference; refine once the install is measured. -->
+  <xacro:property name="garmin_sidescan_x" value="${mbes_x + 0.5}" />
+  <xacro:property name="garmin_sidescan_y" value="${mbes_y}" />
+  <xacro:property name="garmin_sidescan_z" value="${mbes_z - 0.01}" />
   <!-- GPS (POSMV-mounted, relative to motion_sensor) -->
   <xacro:property name="gps_x" value="-0.953" />
@@ -126,4 +133,8 @@
   <xacro:ben_mbes name="mbes"
     x="${mru_x + mbes_x}" y="${mru_y + mbes_y}" z="${mru_z + mbes_z}"/>
+  <xacro:include filename="$(find ben_description)/urdf/sensors/garmin_sidescan.xacro" />
+  <xacro:ben_garmin_sidescan name="garmin_sidescan"
+    x="${mru_x + garmin_sidescan_x}" y="${mru_y + garmin_sidescan_y}"
+    z="${mru_z + garmin_sidescan_z}"/>
   <!-- POSMV-mounted sensors (positions relative to motion_sensor) -->
   <xacro:include filename="$(find ben_description)/urdf/sensors/oem_gps.xacro" />

Commit message: Revert "Add Garmin sidescan TF frames (placeholder geometry) (closes #13)"
This reverts commit d732415eeb63249d5d17684671409521d7628131.

File: urdf/ben_mesh.xacro (robot description, xacro)
@@ -57,11 +57,4 @@
   <xacro:property name="mbes_y" value="0.0" />
   <xacro:property name="mbes_z" value="-0.4" />
-  <!-- Garmin GCV-20 sidescan (hull-mounted, relative to MRU).
-       PLACEHOLDER: ~0.5 m forward of the MBES, glued to the hull with the
-       transducer faces ~1 cm below it. Anchored to the MBES offsets so it
-       tracks the same hull reference; refine once the install is measured. -->
-  <xacro:property name="garmin_sidescan_x" value="${mbes_x + 0.5}" />
-  <xacro:property name="garmin_sidescan_y" value="${mbes_y}" />
-  <xacro:property name="garmin_sidescan_z" value="${mbes_z - 0.01}" />
   <!-- GPS (POSMV-mounted, relative to motion_sensor) -->
   <xacro:property name="gps_x" value="-0.953" />
@@ -133,8 +126,4 @@
   <xacro:ben_mbes name="mbes"
     x="${mru_x + mbes_x}" y="${mru_y + mbes_y}" z="${mru_z + mbes_z}"/>
-  <xacro:include filename="$(find ben_description)/urdf/sensors/garmin_sidescan.xacro" />
-  <xacro:ben_garmin_sidescan name="garmin_sidescan"
-    x="${mru_x + garmin_sidescan_x}" y="${mru_y + garmin_sidescan_y}"
-    z="${mru_z + garmin_sidescan_z}"/>
   <!-- POSMV-mounted sensors (positions relative to motion_sensor) -->
   <xacro:include filename="$(find ben_description)/urdf/sensors/oem_gps.xacro" />
